File: CoCo2VideoMod.kicad_sch (KiCad schematic)
At the start: 22 parts, among them J1 Conn_01x05, J2 Conn_01x03

Commit message: added local symbol library
Parts:
- U?: symbol RivenHexagon:MC1372P -> TRS-80:MC1372P
Changed lines of the file:
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@@
     (pin "3")
   )
-  (symbol (lib_id "RivenHexagon:MC1372P") (at 127 77.47 0) (unit 1)
+  (symbol (lib_id "TRS-80:MC1372P") (at 127 77.47 0) (unit 1)
     (in_bom yes) (on_board yes)
     (property "Reference" "U?" (id 0) (at 129.54 78.74 90)
